File: scratch-rp2040/scratch-rp2040.kicad_sch (KiCad schematic)
At the start: 32 parts, among them P1 USB_C_Plug_USB2.0, SW1 SW_SPST, SW2 SW_SPST, SW3 SW_SPST, SW4 SW_SPST, SW5 SW_SPST, SW6 SW_SPST, SW7 SW_SPST, U1 RP2040, U2 NCP1117-3.3_SOT223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

Commit message: parts placed
Parts:
- P1: footprint Connector_USB:USB_C_Receptacle_GCT_USB4135-GF-A_6P_TopMnt_Horizontal -> Connector_USB:USB_C_Receptacle_G-Switch_GT-USB-7010ASV
Other:
- note added: "Make sure R1 and R2 are close to RP2040"
- note removed: "Make sure R3 and R4 are close to RP2040"
Changed lines of the file:
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@@
     (stroke (width 0) (type default))
   )
-  (text "Make sure R3 and R4 are close to RP2040\n" (at 201.93 71.12 0)
+  (text "Make sure R1 and R2 are close to RP2040\n" (at 201.93 71.12 0)
     (effects (font (size 1.27 1.27)) (justify left bottom))
   )
@@
       (effects (font (size 1.27 1.27)))
     )
-    (property "Footprint" "Connector_USB:USB_C_Receptacle_GCT_USB4135-GF-A_6P_TopMnt_Horizontal" (at 214.63 97.79 0)
-      (effects (font (size 1.27 1.27)) hide)
-    )
+    (property "Footprint" "Connector_USB:USB_C_Receptacle_G-Switch_GT-USB-7010ASV" (at 214.63 97.79 0)
+      (effects (font (size 1.27 1.27)) hide)
+    )
